File: _autosave-hellen121vag.kicad_sch (KiCad schematic)
At the start: 113 parts, among them J1 USB_B_Mini, J10 AudioJack_THR, J2 Conn_01x01, J3 Conn_01x01, J4 Conn_01x01, J5 Conn_01x01, J6 Conn_01x01, J7 Conn_01x08, J8 Conn_01x06, M1 Module-knock-0.2, M11 Module-vr-discrete-0.4, M2 Module-wbo-0.5, M3 mega-mcu144-0.1, M5 Module-knock-0.2, M6 Module-output-0.3, M7 Module-ign8-0.2, M8 Module-power_12and5V-0.1, M9 Module-wbo-0.5, P1 368255-2, P10 Pad, P11 Pad, P12 Pad, P13 Pad, P14 Pad, P15 Pad, P16 Pad, P17 Pad, P2 Pad, P20 Pad, P28 Pad, P3 Pad, P4 Pad, P40 Pad, P41 Pad, P43 Pad, P44 Pad, P45 Pad, P46 Pad, P48 Pad, P49 Pad, P5 Pad, P56 Pad, P6 Pad, P61 Pad, P63 Pad, P64 Pad, P66 Pad, P67 Pad, P68 Pad, P69 Pad, P7 Pad, P74 Pad, P8 Pad, P80 Pad, P9 Pad, U1 L6205PD, U3 MCP6002-xSN

Commit message: dfd
Parts:
- removed BT1: BATTERY_CR2032, Battery:BatteryHolder_Keystone_1060_1x2032, symbol art-electro-power:BATTERY_CR2032
- removed C1, C16, C2: 100n, hellen-one-common:C0603, symbol hellen-one-common:Cap
- removed C10, C11, C12, C13, C14, C7, C8, C9: 10u, Capacitor_SMD:C_0805_2012Metric, symbol hellen-one-common:Cap
- removed C17: 10u, hellen-one-common:C0603, symbol hellen-one-common:Cap
- removed C3: 220n, hellen-one-common:C0603, symbol hellen-one-common:Cap
- removed C4: 10n, hellen-one-common:C0603, symbol hellen-one-common:Cap
- removed C5: 5.6n, hellen-one-common:C0603, symbol hellen-one-common:Cap
- removed D1, D2, D3, D5, D9: 1N4148WS, hellen-one-common:SOD-323, symbol hellen-one-common:1N4148WS
- removed D10, D11, D12, D13, D14: B5819W, Diode_SMD:D_SOD-123, symbol hellen-one-common:1N4148WS
- removed D4, D6, D7, D8: LED-GREEN-0805, hellen-one-common:LED-0805, symbol hellen-one-common:LED
- removed F1, F2: Fuse-Pad-Pad, hellen-one-common:PAD-1206-PAD, symbol hellen-one-common:Fuse-Pad-Pad
- removed G1, G2, G3, G5: PROTO_AREA, hellen-one-common:PROTO_AREA, symbol hellen-one-common:PROTO_AREA
- removed G4: DISCLAIMER, rusefi_lib:Off_Road_Disclaimer, symbol Off_Road_Disclaimer:Disclaimer
- removed G6: LOGO, hellen-one-common:LOGO, symbol hellen-one-common:LOGO
- removed G7: LOGO, rusefi_lib:LOGO, symbol logo:LOGO
- removed J1: USB_B_Mini, hellen-one-common:USB-MINI-B-VERTICAL, symbol hellen-one-common:USB_B_Mini
- removed J10: AudioJack_THR, hellen-one-common:Jack_3.5mm_PJ-3250-5A, symbol hellen-one-common:AudioJack_THR
- removed J2, J3, J4, J5, J6: Conn_01x01, TestPoint:TestPoint_Pad_D2.0mm, symbol Connector_Generic:Conn_01x01
- removed J7: Conn_01x08, Connector_PinHeader_2.54mm:PinHeader_1x08_P2.54mm_Vertical, symbol Connector_Generic:Conn_01x08
- removed J8: Conn_01x06, Connector_PinHeader_2.54mm:PinHeader_1x06_P2.54mm_Vertical, symbol Connector_Generic:Conn_01x06
- removed M1, M5: Module-knock-0.2, hellen-one-knock-0.2:knock, symbol hellen-one-knock-0.2:Module-knock-0.2
- removed M11: Module-vr-discrete-0.4, hellen-one-vr-discrete-0.4:vr-discrete, symbol vr-discrete-0.4:Module-vr-discrete-0.4
- removed M2, M9: Module-wbo-0.5, hellen-one-wbo-0.5:wbo, symbol hellen-one-wbo-0.5:Module-wbo-0.5
- removed M3: mega-mcu144-0.1, hellen-one-mega-mcu144-0.1:mega-mcu144, symbol mega-mcu144-0.1:mega-mcu144-0.1
- removed M6: Module-output-0.3, hellen-one-output-0.3:output, symbol hellen-one-output-0.3:Module-output-0.3
- removed M7: Module-ign8-0.2, hellen-one-ign8-0.2:ign8, symbol hellen-one-ign8-0.2:Module-ign8-0.2
- removed M8: Module-power_12and5V-0.1, hellen-one-power_12and5V-0.1:power_12and5V, symbol power_12and5V-0.1:Module-power_12and5V-0.1
- removed P10, P11, P12, P13, P14, P15, P16, P17, P2, P20, P28, P3, P4, P40, P41, P43, P44, P45, P46, P48, P49, P5, P56, P6, P61, P63, P64, P66, P67, P68, P69, P7, P74, P8, P80, P9: Pad, hellen-one-common:PAD-TH, symbol hellen-one-common:Pad
- removed R1: 100, hellen-one-common:R0603, symbol hellen-one-common:Res
- removed R10, R11, R12, R13, R2, R3, R4, R8, R9: Jumper-Pad-Pad, hellen-one-common:PAD-0805-PAD, symbol hellen-one-common:Jumper-Pad-Pad
- removed R16, R17: 5.1k, hellen-one-common:R0603, symbol hellen-one-common:Res
- removed R20: 1.6k, hellen-one-common:R0603, symbol hellen-one-common:Res
- removed R21: 750, hellen-one-common:R0603, symbol hellen-one-common:Res
- removed R22: 10k, hellen-one-common:R0603, symbol hellen-one-common:Res
- removed R23: 0, hellen-one-common:R0603, symbol hellen-one-common:Res
- removed R5: 100k, hellen-one-common:R0603, symbol hellen-one-common:Res
- removed U1: L6205PD, hellen-one-common:SO20POWER, symbol hellen-one-common:L6205PD
- removed U3: MCP6002-xSN, Package_SO:SOIC-8_3.9x4.9mm_P1.27mm, symbol Amplifier_Operational:MCP6002-xSN
- P1: footprint hellen121vag:368255-2 -> 368255-2:368255-2
Connections:
- removed net +5VP: P1.53, P1.72, P1.73, P1.83, P1.98
- net +ETB_OUT: no longer names the net of P1.117
- net -ETB_OUT: no longer names the net of P1.118
- net CAN+: no longer names the net of P1.60
- net CAN-: no longer names the net of P1.58
- removed net GND: P1.1, P1.2, P1.32, P1.59
- removed net GNDA: P1.108, P1.27, P1.33, P1.36, P1.50, P1.91, P1.99
- net IN_AFR: no longer names the net of P1.14
- net IN_CAM1: no longer names the net of P1.86
- net IN_CAM2: no longer names the net of P1.87
- net IN_CLT: no longer names the net of P1.93
- net IN_CRANK+: no longer names the net of P1.82
- net IN_CRANK-: no longer names the net of P1.90
- net IN_D1: no longer names the net of P1.55
- net IN_D2: no longer names the net of P1.57
- net IN_D3: no longer names the net of P1.75
- net IN_D4: no longer names the net of P1.76
- net IN_IAT: no longer names the net of P1.26
- net IN_IAT: no longer P1.85
- net IN_KNOCK1_RAW: no longer names the net of P1.106
- net IN_MAF: no longer names the net of P1.29
- net IN_MAP2: no longer names the net of P1.101
- net IN_PPS1: no longer names the net of P1.34
- net IN_PPS2: no longer names the net of P1.35
- net IN_RES1: no longer names the net of P1.38
- net IN_RES2: no longer names the net of P1.39
- net IN_TPS1: no longer names the net of P1.92
- net IN_TPS2: no longer names the net of P1.84
- net IN_VSS: no longer names the net of P1.54
- net LSU_HEAT-: no longer names the net of P1.5
- net OUT_CHECK_ENGINE: no longer names the net of P1.47
- net OUT_FUEL_CONSUM: no longer names the net of P1.81
- net OUT_FUEL_PUMP_RELAY: no longer names the net of P1.65
- net OUT_IDLE: no longer names the net of P1.105
- net OUT_IGN1: no longer names the net of P1.102
- net OUT_IGN2: no longer names the net of P1.7
- net OUT_IGN3: no longer names the net of P1.111
- net OUT_IGN4: no longer names the net of P1.94
- net OUT_IGN5: no longer names the net of P1.103
- net OUT_IGN6: no longer names the net of P1.110
- net OUT_IGN7: no longer names the net of P1.8
- net OUT_IGN8: no longer names the net of P1.95
- net OUT_INJ1: no longer names the net of P1.96
- net OUT_INJ2: no longer names the net of P1.89
- net OUT_INJ3: no longer names the net of P1.97
- net OUT_INJ4: no longer names the net of P1.88
- net OUT_INJ5: no longer names the net of P1.113
- net OUT_INJ6: no longer names the net of P1.112
- net OUT_INJ7: no longer names the net of P1.19
- net OUT_INJ8: no longer names the net of P1.24
- net OUT_VVT1_1: no longer names the net of P1.22
- net OUT_VVT1_2: no longer names the net of P1.115
- net OUT_VVT2_B1: no longer names the net of P1.18
- net OUT_VVT2_B2: no longer names the net of P1.120
- net OUT_WASTEGATE: no longer names the net of P1.104
- net V12_PERM: no longer names the net of P1.62
- no-connect marks 70 -> 0
Other:
- note removed: "#1"
- note removed: "Analog inputs (sensors)"
- note removed: "Board info"
- note removed: "Bus types"
- note removed: "Discrete inputs"
- note removed: "ETB driver"
- note removed: "General purpose bus"
- note removed: "Ignition"
- note removed: "Injection"
- note removed: "LEDs"
- note removed: "Ouputs"
- note removed: "Power"
- note removed: "Prototype areas"
- note removed: "TODO: knock 2"
- note removed: "http://rusefi.com/s/hellen121vag"
- note removed: "to ETB driver"
