File: hellen121vag.kicad_pcb (KiCad board)
At the start: 4 copper layers, 164 x 118 mm, 129 parts, among them J1 USB_B_Mini, J10 AudioJack_THR, J2 Conn_01x01, J3 Conn_01x01, J4 Conn_01x01, J5 Conn_01x01, J6 Conn_01x01, J7 Conn_01x08, J8 Conn_01x06, M1 Module-can-0.1, M10 Module-can-0.1, M11 Module-vr-discrete-0.1, M2 Module-power5-0.2, M3 Module-mcu-0.7, M4 Module-input-0.1, M5 Module-knock-0.1, M6 Module-output-0.3, M7 Module-ign8-0.2, M8 Module-power12-0.2, M9 Module-wbo-0.3, P1 368255-2, P10 Pad, P11 Pad, P12 Pad, P13 Pad, P14 Pad, P15 Pad, P16 Pad, P17 Pad, P2 Pad, P20 Pad, P28 Pad, P3 Pad, P4 Pad, P40 Pad, P41 Pad, P43 Pad, P44 Pad, P45 Pad, P46 Pad, P48 Pad, P49 Pad, P5 Pad, P56 Pad, P6 Pad, P61 Pad, P63 Pad, P64 Pad, P66 Pad, P67 Pad, P68 Pad, P69 Pad, P7 Pad, P74 Pad, P8 Pad, P80 Pad, P9 Pad, U1 L6205PD, U2 LPS25HB, U3 MCP6002-xSN, U4 TLS115_SOIC, U5 TLS115_SON

Commit message: gyr
Parts:
- removed M3: Module-mcu-0.7, hellen-one-mcu-0.7:mcu
- added M1: Module-knock-0.2, hellen-one-knock-0.2:knock, F.Cu at (173.0, -1.40)
- added M2: Module-wbo-0.5, hellen-one-wbo-0.5:wbo, F.Cu at (45.8, 9.07)
- added M5: Module-knock-0.2, hellen-one-knock-0.2:knock, F.Cu at (74.7, 2.83)
- added M9: Module-wbo-0.5, hellen-one-wbo-0.5:wbo, F.Cu at (45.8, 24.4)
- moved U4 36.1 mm to (57.2, 63.9)
- moved C18 36.1 mm to (62.4, 70.2)
- moved C19 36.1 mm to (62.4, 68.2)
- moved U5 36.1 mm to (58.0, 69.6)
Connections:
- J8 pad 1: Net-(J8-Pad1) -> Net-(J8-Pin_1)
- J8 pad 2: Net-(J8-Pad2) -> Net-(J8-Pin_2)
- J8 pad 4: Net-(J8-Pad4) -> Net-(J8-Pin_4)
- J8 pad 5: Net-(J8-Pad5) -> Net-(J8-Pin_5)

Commit message: dfd
Parts:
- removed BT1: BATTERY_CR2032, Battery:BatteryHolder_Keystone_1060_1x2032
- removed C1, C15, C16, C2, C6: 100n, hellen-one-common:C0603
- removed C10, C11, C12, C13, C14, C7, C8, C9: 10u, Capacitor_SMD:C_0805_2012Metric
- removed C17: 10u, hellen-one-common:C0603
- removed C18, C19: 1u, hellen-one-common:C0603
- removed C3: 220n, hellen-one-common:C0603
- removed C4: 10n, hellen-one-common:C0603
- removed C5: 5.6n, hellen-one-common:C0603
- removed D1, D2, D3, D5, D9: 1N4148WS, hellen-one-common:SOD-323
- removed D10, D11, D12, D13, D14: B5819W, Diode_SMD:D_SOD-123
- removed D4, D6, D7, D8: LED-GREEN-0805, hellen-one-common:LED-0805
- removed F1, F2: Fuse-Pad-Pad, hellen-one-common:PAD-1206-PAD
- removed G***, G6: LOGO, hellen-one-common:LOGO
- removed G1, G2, G3, G5: PROTO_AREA, hellen-one-common:PROTO_AREA
- removed G7: LOGO, rusefi_lib:LOGO
- removed J1: USB_B_Mini, hellen-one-common:USB-MINI-B-VERTICAL
- removed J10: AudioJack_THR, hellen-one-common:Jack_3.5mm_PJ-3250-5A
- removed J2, J3, J4, J5, J6: Conn_01x01, TestPoint:TestPoint_Pad_D2.0mm
- removed J7: Conn_01x08, Connector_PinHeader_2.54mm:PinHeader_1x08_P2.54mm_Vertical
- removed J8: Conn_01x06, Connector_PinHeader_2.54mm:PinHeader_1x06_P2.54mm_Vertical
- removed M1, M10: Module-can-0.1, hellen-one-can-0.1:can
- removed M1, M5: Module-knock-0.2, hellen-one-knock-0.2:knock
- removed M11: Module-vr-discrete-0.1, hellen-one-vr-discrete-0.1:vr-discrete
- removed M2, M9: Module-wbo-0.5, hellen-one-wbo-0.5:wbo
- removed M2: Module-power5-0.2, hellen-one-power5-0.2:power5
- removed M4: Module-input-0.1, hellen-one-input-0.1:input
- removed M5: Module-knock-0.1, hellen-one-knock-0.1:knock
- removed M6: Module-output-0.3, hellen-one-output-0.3:output
- removed M7: Module-ign8-0.2, hellen-one-ign8-0.2:ign8
- removed M8: Module-power12-0.2, hellen-one-power12-0.2:power12
- removed M9: Module-wbo-0.3, hellen-one-wbo-0.3:wbo
- removed P10, P11, P12, P13, P14, P15, P16, P17, P2, P20, P28, P3, P4, P40, P41, P43, P44, P45, P46, P48, P49, P5, P56, P6, P61, P63, P64, P66, P67, P68, P69, P7, P74, P8, P80, P9: Pad, hellen-one-common:PAD-TH
- removed R1: 100, hellen-one-common:R0603
- removed R10, R11, R12, R13, R2, R3, R4, R8, R9: Jumper-Pad-Pad, hellen-one-common:PAD-0805-PAD
- removed R16, R17: 5.1k, hellen-one-common:R0603
- removed R18, R19: 4.7k, hellen-one-common:R0603
- removed R20: 1.6k, hellen-one-common:R0603
- removed R21: 750, hellen-one-common:R0603
- removed R22: 10k, hellen-one-common:R0603
- removed R23: 0, hellen-one-common:R0603
- removed R5: 100k, hellen-one-common:R0603
- removed R6, R7: 2.7k, hellen-one-common:R0603
- removed S1, S2: Button_SPST, hellen-one-common:SMD-2_2.9x3.9x1.7
- removed U1: L6205PD, hellen-one-common:SO20POWER
- removed U2: LPS25HB, Package_LGA:ST_HLGA-10_2.5x2.5mm_P0.6mm_LayoutBorder3x2y
- removed U3: MCP6002-xSN, Package_SO:SOIC-8_3.9x4.9mm_P1.27mm
- removed U4: TLS115_SOIC, kicad6-libraries:PG-DSO-8-43_VIA
- removed U5: TLS115_SON, Package_SON:HVSON-8-1EP_3x3mm_P0.65mm_EP1.6x2.4mm
- P1: footprint hellen121vag:368255-2 -> 368255-2:368255-2
Connections:
- P1 pad 1: GND -> unconnected-(P1-Pad1)
- P1 pad 10: Net-(P10-Pin_1) -> unconnected-(P1-Pad10)
- P1 pad 101: /IN_MAP2 -> unconnected-(P1-Pad101)
- P1 pad 102: /OUT_IGN1 -> unconnected-(P1-Pad102)
- P1 pad 103: /OUT_IGN5 -> unconnected-(P1-Pad103)
- P1 pad 104: /OUT_WASTEGATE -> unconnected-(P1-Pad104)
- P1 pad 105: /OUT_IDLE -> unconnected-(P1-Pad105)
- P1 pad 106: /IN_KNOCK1_RAW -> unconnected-(P1-Pad106)
- P1 pad 108: GNDA -> unconnected-(P1-Pad108)
- P1 pad 11: Net-(P11-Pin_1) -> unconnected-(P1-Pad11)
- P1 pad 110: /OUT_IGN6 -> unconnected-(P1-Pad110)
- P1 pad 111: /OUT_IGN3 -> unconnected-(P1-Pad111)
- P1 pad 112: /OUT_INJ6 -> unconnected-(P1-Pad112)
- P1 pad 113: /OUT_INJ5 -> unconnected-(P1-Pad113)
- P1 pad 115: /OUT_VVT1_2 -> unconnected-(P1-Pad115)
- P1 pad 117: /+ETB_OUT -> unconnected-(P1-Pad117)
- P1 pad 118: /-ETB_OUT -> unconnected-(P1-Pad118)
- P1 pad 12: Net-(P12-Pin_1) -> unconnected-(P1-Pad12)
- P1 pad 120: /OUT_VVT2_B2 -> unconnected-(P1-Pad120)
- P1 pad 121: Net-(F2-Pad1) -> unconnected-(P1-Pad121)
- P1 pad 13: Net-(P13-Pin_1) -> unconnected-(P1-Pad13)
- P1 pad 14: /IN_AFR -> unconnected-(P1-Pad14)
- P1 pad 17: Net-(P17-Pin_1) -> unconnected-(P1-Pad17)
- P1 pad 18: /OUT_VVT2_B1 -> unconnected-(P1-Pad18)
- P1 pad 19: /OUT_INJ7 -> unconnected-(P1-Pad19)
- P1 pad 2: GND -> unconnected-(P1-Pad2)
- P1 pad 20: Net-(P20-Pin_1) -> unconnected-(P1-Pad20)
- P1 pad 21: Net-(P1-Pad21) -> unconnected-(P1-Pad21)
- P1 pad 22: /OUT_VVT1_1 -> unconnected-(P1-Pad22)
- P1 pad 23: Net-(P1-Pad23) -> unconnected-(P1-Pad23)
- P1 pad 24: /OUT_INJ8 -> unconnected-(P1-Pad24)
- P1 pad 26: /IN_IAT -> unconnected-(P1-Pad26)
- P1 pad 27: GNDA -> unconnected-(P1-Pad27)
- P1 pad 28: Net-(P28-Pin_1) -> unconnected-(P1-Pad28)
- P1 pad 29: /IN_MAF -> unconnected-(P1-Pad29)
- P1 pad 3: Net-(F1-Pad1) -> unconnected-(P1-Pad3)
- P1 pad 32: GND -> unconnected-(P1-Pad32)
- P1 pad 33: GNDA -> unconnected-(P1-Pad33)
- P1 pad 34: /IN_PPS1 -> unconnected-(P1-Pad34)
- P1 pad 35: /IN_PPS2 -> unconnected-(P1-Pad35)
- P1 pad 36: GNDA -> unconnected-(P1-Pad36)
- P1 pad 37: Net-(P1-Pad37) -> unconnected-(P1-Pad37)
- P1 pad 38: /IN_RES1 -> unconnected-(P1-Pad38)
- P1 pad 39: /IN_RES2 -> unconnected-(P1-Pad39)
- P1 pad 40: Net-(P40-Pin_1) -> unconnected-(P1-Pad40)
- P1 pad 41: Net-(P41-Pin_1) -> unconnected-(P1-Pad41)
- P1 pad 43: Net-(P43-Pin_1) -> unconnected-(P1-Pad43)
- P1 pad 44: Net-(P44-Pin_1) -> unconnected-(P1-Pad44)
- P1 pad 45: Net-(P45-Pin_1) -> unconnected-(P1-Pad45)
- P1 pad 46: Net-(P46-Pin_1) -> unconnected-(P1-Pad46)
- P1 pad 47: /OUT_CHECK_ENGINE -> unconnected-(P1-Pad47)
- P1 pad 48: Net-(P48-Pin_1) -> unconnected-(P1-Pad48)
- P1 pad 49: Net-(P49-Pin_1) -> unconnected-(P1-Pad49)
- P1 pad 5: /LSU_HEAT- -> unconnected-(P1-Pad5)
- P1 pad 50: GNDA -> unconnected-(P1-Pad50)
- P1 pad 51: Net-(P1-Pad51) -> unconnected-(P1-Pad51)
- P1 pad 52: Net-(P1-Pad52) -> unconnected-(P1-Pad52)
- P1 pad 53: +5VP -> unconnected-(P1-Pad53)
- P1 pad 54: /IN_VSS -> unconnected-(P1-Pad54)
- P1 pad 55: /IN_D1 -> unconnected-(P1-Pad55)
- P1 pad 56: Net-(P56-Pin_1) -> unconnected-(P1-Pad56)
- P1 pad 57: /IN_D2 -> unconnected-(P1-Pad57)
- P1 pad 58: /CAN- -> unconnected-(P1-Pad58)
- P1 pad 59: GND -> unconnected-(P1-Pad59)
- P1 pad 60: /CAN+ -> unconnected-(P1-Pad60)
- P1 pad 61: Net-(P61-Pin_1) -> unconnected-(P1-Pad61)
- P1 pad 62: /V12_PERM -> unconnected-(P1-Pad62)
- P1 pad 63: Net-(P63-Pin_1) -> unconnected-(P1-Pad63)
- P1 pad 64: Net-(P64-Pin_1) -> unconnected-(P1-Pad64)
- P1 pad 65: /OUT_FUEL_PUMP_RELAY -> unconnected-(P1-Pad65)
- P1 pad 66: Net-(P66-Pin_1) -> unconnected-(P1-Pad66)
- P1 pad 67: Net-(P67-Pin_1) -> unconnected-(P1-Pad67)
- P1 pad 68: Net-(P68-Pin_1) -> unconnected-(P1-Pad68)
- P1 pad 69: Net-(P69-Pin_1) -> unconnected-(P1-Pad69)
- P1 pad 7: /OUT_IGN2 -> unconnected-(P1-Pad7)
- P1 pad 70: Net-(P1-Pad70) -> unconnected-(P1-Pad70)
- P1 pad 71: Net-(P1-Pad71) -> unconnected-(P1-Pad71)
- P1 pad 72: +5VP -> unconnected-(P1-Pad72)
- P1 pad 73: +5VP -> unconnected-(P1-Pad73)
- P1 pad 74: Net-(P74-Pin_1) -> unconnected-(P1-Pad74)
- P1 pad 75: /IN_D3 -> unconnected-(P1-Pad75)
- P1 pad 76: /IN_D4 -> unconnected-(P1-Pad76)
- P1 pad 8: /OUT_IGN7 -> unconnected-(P1-Pad8)
- P1 pad 80: Net-(P80-Pin_1) -> unconnected-(P1-Pad80)
- P1 pad 81: /OUT_FUEL_CONSUM -> unconnected-(P1-Pad81)
- P1 pad 82: /IN_CRANK+ -> unconnected-(P1-Pad82)
- P1 pad 83: +5VP -> unconnected-(P1-Pad83)
- P1 pad 84: /IN_TPS2 -> unconnected-(P1-Pad84)
- P1 pad 85: /IN_IAT -> unconnected-(P1-Pad85)
- P1 pad 86: /IN_CAM1 -> unconnected-(P1-Pad86)
- P1 pad 87: /IN_CAM2 -> unconnected-(P1-Pad87)
- P1 pad 88: /OUT_INJ4 -> unconnected-(P1-Pad88)
- P1 pad 89: /OUT_INJ2 -> unconnected-(P1-Pad89)
- P1 pad 9: Net-(P9-Pin_1) -> unconnected-(P1-Pad9)
- P1 pad 90: /IN_CRANK- -> unconnected-(P1-Pad90)
- P1 pad 91: GNDA -> unconnected-(P1-Pad91)
- P1 pad 92: /IN_TPS1 -> unconnected-(P1-Pad92)
- P1 pad 93: /IN_CLT -> unconnected-(P1-Pad93)
- P1 pad 94: /OUT_IGN4 -> unconnected-(P1-Pad94)
- P1 pad 95: /OUT_IGN8 -> unconnected-(P1-Pad95)
- P1 pad 96: /OUT_INJ1 -> unconnected-(P1-Pad96)
- P1 pad 97: /OUT_INJ3 -> unconnected-(P1-Pad97)
- P1 pad 98: +5VP -> unconnected-(P1-Pad98)
- P1 pad 99: GNDA -> unconnected-(P1-Pad99)
Routing:
- net +12V_RAW: track 567.8 -> 0.00 mm, vias 18 -> 0
- net +5V: track 359.2 -> 0.00 mm, vias 4 -> 0
- net +3V3: track 198.6 -> 0.00 mm, vias 4 -> 0
- net /OUT_IGN1: track 181.1 -> 0.00 mm, vias 2 -> 0
- net /OUT_IGN3: track 177.7 -> 0.00 mm, vias 2 -> 0
- net /OUT_IGN5: track 173.6 -> 0.00 mm, vias 1 -> 0
- net /OUT_IGN6: track 172.1 -> 0.00 mm, vias 2 -> 0
- net /OUT_IGN4: track 171.5 -> 0.00 mm, vias 2 -> 0
- net /IN_VIGN: track 171.1 -> 0.00 mm, vias 1 -> 0
- net /OUT_IGN8: track 161.5 -> 0.00 mm, vias 1 -> 0
- net Net-(F1-Pad1): track 156.2 -> 0.00 mm, vias 1 -> 0
- net /OUT_IGN2: track 155.4 -> 0.00 mm, vias 2 -> 0
- net /OUT_IGN7: track 135.0 -> 0.00 mm, vias 2 -> 0
- net /OUT_FUEL_CONSUM: track 135.0 -> 0.00 mm, vias 3 -> 0
- net /OUT_VVT2_B1: track 124.6 -> 0.00 mm, vias 3 -> 0
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- added copper zone on B.Cu, net unconnected-(P1-Pad59)
- added copper zone on F.Cu, net unconnected-(P1-Pad59)
- removed copper zone on B.Cu, net /OUT_INJ2
- removed copper zone on B.Cu, net GND
- removed copper zone on F.Cu, net GND
- removed copper zone on In1.Cu, net GND
- removed copper zone on B.Cu, net Net-(J1-GND)
- removed copper zone on F.Cu, net Net-(J1-GND)
Other:
- board text removed: "+12"
- board text removed: "+3.3"
- board text removed: "+5"
- board text removed: "1"
- board text removed: "10"
- board text removed: "100"
- board text removed: "101"
- board text removed: "102"
- board text removed: "103"
- board text removed: "104"
- board text removed: "105"
- board text removed: "106"
- board text removed: "11"
- board text removed: "112"
- board text removed: "113"
- board text removed: "114"
- board text removed: "115"
- board text removed: "116"
- board text removed: "117"
- board text removed: "118"
- board text removed: "119"
- board text removed: "12"
- board text removed: "120"
- board text removed: "121"
- board text removed: "12V SRC"
- board text removed: "13"
- board text removed: "14"
- board text removed: "15"
- board text removed: "16"
- board text removed: "17"
- board text removed: "18"
- board text removed: "19"
- board text removed: "2"
- board text removed: "20"
- board text removed: "21"
- board text removed: "22"
- board text removed: "23"
- board text removed: "24"
- board text removed: "25"
- board text removed: "26"
- board text removed: "27"
- board text removed: "28"
- board text removed: "29"
- board text removed: "3"
- board text removed: "3.3"
- board text removed: "30"
- board text removed: "31"
- board text removed: "32"
- board text removed: "33"
- board text removed: "34"
- board text removed: "35"
- board text removed: "36"
- board text removed: "37"
- board text removed: "38"
- board text removed: "39"
- board text removed: "4"
- board text removed: "40"
- board text removed: "41"
- board text removed: "42"
- board text removed: "43"
- board text removed: "44"
- board text removed: "45"
- board text removed: "46"
- board text removed: "47"
- board text removed: "48"
- board text removed: "49"
- board text removed: "5"
- board text removed: "50"
- board text removed: "51"
- board text removed: "52"
- board text removed: "53"
- board text removed: "54"
- board text removed: "55"
- board text removed: "56"
- board text removed: "57"
- board text removed: "58"
- board text removed: "59"
- board text removed: "6"
- board text removed: "60"
- board text removed: "61"
- board text removed: "62"
- board text removed: "63"
- board text removed: "64"
- board text removed: "65"
- board text removed: "66"
- board text removed: "67"
- board text removed: "68"
- board text removed: "69"
- board text removed: "7"
- board text removed: "70"
- board text removed: "71"
- board text removed: "72"
- board text removed: "73"
- board text removed: "74"
- board text removed: "75"
- board text removed: "76"
- board text removed: "77"
- board text removed: "78"
- board text removed: "79"
- board text removed: "8"
- board text removed: "80"
- board text removed: "81"
- board text removed: "82"
- board text removed: "83"
- board text removed: "84"
- board text removed: "85"
- board text removed: "86"
- board text removed: "87"
- board text removed: "88"
- board text removed: "89"
- board text removed: "9"
- board text removed: "90"
- board text removed: "91"
- board text removed: "92"
- board text removed: "93"
- board text removed: "94"
- board text removed: "95"
- board text removed: "96"
- board text removed: "97"
- board text removed: "98"
- board text removed: "99"
- board text removed: "<- Knock audio"
- board text removed: "Always looking for C/C++/PHP/Java developers https://rusefi.com/s/mission"
- board text removed: "Baro"
- board text removed: "CLK"
- board text removed: "DIO"
- board text removed: "G"
- board text removed: "GND"
- board text removed: "Hellen121vag"
- board text removed: "PROG"
- board text removed: "RESET"
- board text removed: "RST"
- board text removed: "SWD WBO"
- board text removed: "Vign"
- board text removed: "http://rusefi.com/s/hellen121vag"
- board text removed: "rev. d"
- board text removed: "© andreika, 2021"
