File: hellen121vag.kicad_pcb (KiCad board)
At the start: 4 copper layers, 164 x 118 mm, 2 parts, among them P1 368255-2

Commit message: ewr
Parts:
- added BT1: CR1220, kicad6-libraries:CR1220-2, B.Cu at (224.3, 311.6)
- added C1: 10u, hellen-one-common:C0805, B.Cu at (136.4, 318.2)
- added C10: 10u, hellen-one-common:C0805, B.Cu at (144.4, 322.2)
- added C11: 100n, hellen-one-common:C0603, F.Cu at (133.9, 319.8)
- added C12: 10n, hellen-one-common:C0603, F.Cu at (133.9, 322.9)
- added C13: 10n, hellen-one-common:C0603, F.Cu at (149.0, 322.2)
- added C14: 10u, hellen-one-common:C0805, B.Cu at (142.9, 327.6)
- added C15: 10u, hellen-one-common:C0805, B.Cu at (144.9, 327.6)
- added C16: 10u, hellen-one-common:C0805, B.Cu at (146.9, 327.6)
- added C17: 10u, hellen-one-common:C0805, B.Cu at (148.9, 327.6)
- added C18: 10u, hellen-one-common:C0805, B.Cu at (150.9, 327.6)
- added C19: 10u, hellen-one-common:C0805, B.Cu at (142.9, 331.6)
- added C2: 10u, hellen-one-common:C0805, B.Cu at (138.4, 318.2)
- added C20: 10u, hellen-one-common:C0805, B.Cu at (144.9, 331.6)
- added C21: 10u, hellen-one-common:C0805, B.Cu at (146.9, 331.6)
- added C22: 10u, hellen-one-common:C0805, B.Cu at (148.9, 331.6)
- added C23: 10u, hellen-one-common:C0805, B.Cu at (150.9, 331.6)
- added C24: 100n, hellen-one-common:C0603, F.Cu at (139.9, 328.1)
- added C25: 10n, hellen-one-common:C0603, F.Cu at (139.9, 331.6)
- added C26: 10n, hellen-one-common:C0603, F.Cu at (155.9, 331.6)
- added C27: 100n, hellen-one-common:C0603, B.Cu at (194.1, 272.0)
- added C28: 10n, hellen-one-common:C0603, B.Cu at (186.1, 254.5)
- added C29: 100n, hellen-one-common:C0603, B.Cu at (187.8, 260.1)
- added C3: 10u, hellen-one-common:C0805, B.Cu at (140.4, 318.2)
- added C30: 10n, hellen-one-common:C0603, B.Cu at (189.5, 254.5)
- added C31: 100n, hellen-one-common:C0603, B.Cu at (191.9, 263.6)
- added C32: 1u, hellen-one-common:C0603, B.Cu at (193.7, 263.6)
- added C33: 100n, hellen-one-common:C0603, B.Cu at (229.3, 303.1)
- added C4: 10u, hellen-one-common:C0805, B.Cu at (142.4, 318.2)
- added C5: 10u, hellen-one-common:C0805, B.Cu at (144.4, 318.2)
- added C6: 10u, hellen-one-common:C0805, B.Cu at (136.4, 322.2)
- added C7: 10u, hellen-one-common:C0805, B.Cu at (138.4, 322.2)
- added C8: 10u, hellen-one-common:C0805, B.Cu at (140.4, 322.2)
- added C9: 10u, hellen-one-common:C0805, B.Cu at (142.4, 322.2)
- added D1: 1N4148WS, hellen-one-common:SOD-323, B.Cu at (220.3, 321.1)
- added D2: B5819W, hellen-one-common:SOD-123, B.Cu at (151.3, 266.6)
- added D3: B5819W, hellen-one-common:SOD-123, F.Cu at (151.3, 260.6)
- added D4: B5819W, hellen-one-common:SOD-123, B.Cu at (151.3, 259.1)
- added D5: B5819W, hellen-one-common:SOD-123, F.Cu at (151.3, 268.1)
- added D8: NUP2105L, Package_TO_SOT_SMD:SOT-23, B.Cu at (187.8, 257.6)
- added F1: 12H1500D, hellen-one-common:PAD-1206-PAD, F.Cu at (155.1, 320.1)
- added F10: 50mA, Fuse:Fuse_0603_1608Metric, B.Cu at (215.5, 304.7)
- added F2: 12H1500D, hellen-one-common:PAD-1206-PAD, F.Cu at (153.3, 314.5)
- added F3: 12H1500D, hellen-one-common:PAD-1206-PAD, F.Cu at (152.9, 320.1)
- added F4: 12H1500D, hellen-one-common:PAD-1206-PAD, F.Cu at (150.7, 320.1)
- added F5: 50mA, Fuse:Fuse_0603_1608Metric, B.Cu at (162.4, 281.7)
- added F6: 50mA, Fuse:Fuse_0603_1608Metric, B.Cu at (162.4, 274.7)
- added F7: 50mA, Fuse:Fuse_0603_1608Metric, B.Cu at (162.5, 288.7)
- added F8: 50mA, Fuse:Fuse_0603_1608Metric, B.Cu at (162.4, 295.7)
- added F9: 50mA, Fuse:Fuse_0603_1608Metric, B.Cu at (162.4, 302.7)
- added G1: RUSEFI_LOGO, kicad6-libraries:rusefi_logo, F.Cu at (221.3, 333.6)
- added G2: LOGO, hellen-one-common:LOGO, F.Cu at (204.3, 331.6)
- added G3: PROTO_AREA, hellen-one-common:PROTO_AREA, F.Cu at (171.8, 287.2)
- added G4: PROTO_AREA, hellen-one-common:PROTO_AREA, F.Cu at (179.4, 287.2)
- added H1: M3, MountingHole:MountingHole_3.2mm_M3_Pad_Via, F.Cu at (135.8, 240.6)
- added H2: M3, MountingHole:MountingHole_3.2mm_M3_Pad_Via, F.Cu at (135.8, 333.6)
- added H3: M3, MountingHole:MountingHole_3.2mm_M3_Pad_Via, F.Cu at (228.8, 333.6)
- added H4: M3, MountingHole:MountingHole_3.2mm_M3_Pad_Via, F.Cu at (228.8, 240.6)
- added J1: Conn_02x02_Odd_Even, Connector_PinSocket_2.54mm:PinSocket_2x02_P2.54mm_Vertical, F.Cu at (221.2, 247.9)
- added J10: 5569-16A2, Connector_Molex:Molex_Mini-Fit_Jr_5569-16A2_2x08_P4.20mm_Horizontal, F.Cu at (192.6, 246.4)
- added J11: Conn_02x02_Odd_Even, Connector_PinSocket_2.54mm:PinSocket_2x02_P2.54mm_Vertical, F.Cu at (212.8, 247.9)
- added J12: Conn_02x02_Odd_Even, Connector_PinSocket_2.54mm:PinSocket_2x02_P2.54mm_Vertical, F.Cu at (204.4, 247.9)
- added J13: Conn_02x02_Odd_Even, Connector_PinSocket_2.54mm:PinSocket_2x02_P2.54mm_Vertical, F.Cu at (196.0, 247.9)
- added J14: Conn_02x02_Odd_Even, Connector_PinSocket_2.54mm:PinSocket_2x02_P2.54mm_Vertical, F.Cu at (146.3, 247.9)
- added J15: Conn_02x02_Odd_Even, Connector_PinSocket_2.54mm:PinSocket_2x02_P2.54mm_Vertical, F.Cu at (154.7, 247.9)
- added J16: Conn_02x02_Odd_Even, Connector_PinSocket_2.54mm:PinSocket_2x02_P2.54mm_Vertical, F.Cu at (163.1, 247.9)
- added J17: Conn_02x02_Odd_Even, Connector_PinSocket_2.54mm:PinSocket_2x02_P2.54mm_Vertical, F.Cu at (171.5, 247.9)
- added J18: Conn_02x02_Odd_Even, Connector_PinSocket_2.54mm:PinSocket_2x02_P2.54mm_Vertical, F.Cu at (145.6, 259.2)
- added J19: Conn_02x02_Odd_Even, Connector_PinSocket_2.54mm:PinSocket_2x02_P2.54mm_Vertical, F.Cu at (145.6, 267.6)
- added J2: 5569-20A2, Connector_Molex:Molex_Mini-Fit_Jr_5569-20A2_2x10_P4.20mm_Horizontal, F.Cu at (142.9, 246.4)
- added J20: Conn_02x02_Odd_Even, Connector_PinSocket_2.54mm:PinSocket_2x02_P2.54mm_Vertical, F.Cu at (145.6, 276.0)
- added J21: Conn_02x02_Odd_Even, Connector_PinSocket_2.54mm:PinSocket_2x02_P2.54mm_Vertical, F.Cu at (145.6, 284.4)
- added J22: Conn_02x02_Odd_Even, Connector_PinSocket_2.54mm:PinSocket_2x02_P2.54mm_Vertical, F.Cu at (145.6, 299.6)
- added J24: Conn_02x02_Odd_Even, Connector_PinSocket_2.54mm:PinSocket_2x02_P2.54mm_Vertical, F.Cu at (221.6, 258.8)
- added J3: 5569-06A2, Connector_Molex:Molex_Mini-Fit_Jr_5569-06A2_2x03_P4.20mm_Horizontal, F.Cu at (223.0, 257.9)
- added J4: 5569-08A2, Connector_Molex:Molex_Mini-Fit_Jr_5569-08A2_2x04_P4.20mm_Horizontal, F.Cu at (141.6, 311.3)
- added J5: 5569-18A2, Connector_Molex:Molex_Mini-Fit_Jr_5569-18A2_2x09_P4.20mm_Horizontal, F.Cu at (141.6, 291.9)
- added J6: Conn_01x06, Connector_PinHeader_2.54mm:PinHeader_1x06_P2.54mm_Vertical, F.Cu at (230.5, 299.2)
- added J7: Conn_01x05_Male, Connector_Molex:Molex_SPOX_5267-05A_1x05_P2.50mm_Vertical, F.Cu at (215.3, 334.1)
- added J8: USB_B_Mini, hellen-one-common:USB-MINI-B-VERTICAL, F.Cu at (190.7, 332.4)
- added J9: USB_C, kicad6-libraries:USB_C, F.Cu at (182.3, 333.1)
- added L1: 470R@100MHz, Inductor_SMD:L_0603_1608Metric, B.Cu at (188.8, 252.1)
- added L2: 470R@100MHz, Inductor_SMD:L_0603_1608Metric, B.Cu at (186.8, 252.1)
- added M1: Module-power_12and5V-0.3, hellen-one-power_12and5V-0.3:power_12and5V, F.Cu at (156.9, 335.9)
- added M2: Module-knock-0.2, hellen-one-knock-0.2:knock, F.Cu at (209.3, 255.0)
- added M3: Module-vr-discrete-0.5, hellen-one-vr-discrete-0.5:vr-discrete, F.Cu at (174.6, 259.7)
- added M4: Module-vr-max9924-0.1, hellen-one-vr-max9924-0.1:vr-max9924, F.Cu at (163.5, 259.7)
- added M5: Module-wbo-0.5, hellen-one-wbo-0.5:wbo, F.Cu at (231.7, 297.5)
- added M6: Module:mega-mcu100/0.3, hellen-one-mega-mcu100-0.3:mega-mcu100, F.Cu at (105.9, 11.6)
- added M7: Module-can-0.1, hellen-one-can-0.1:can, F.Cu at (162.9, 282.5)
- added P1: Pad, hellen-one-common:PAD-TH, F.Cu at (164.3, 279.6)
- added P15: Pad, hellen-one-common:PAD-TH, F.Cu at (137.8, 325.6)
- added P16: Pad, hellen-one-common:PAD-TH, F.Cu at (140.4, 325.6)
- added P17: Pad, hellen-one-common:PAD-TH, F.Cu at (135.3, 325.6)
- added P18: Pad, hellen-one-common:PAD-TH, F.Cu at (155.3, 326.1)
- added P2: Pad, hellen-one-common:PAD-TH, F.Cu at (167.2, 279.6)
- added P3: Pad, hellen-one-common:PAD-TH, F.Cu at (194.8, 334.6)
- added P4: Pad, hellen-one-common:PAD-TH, F.Cu at (194.8, 329.6)
- added P5: Pad, hellen-one-common:PAD-TH, F.Cu at (173.9, 291.1)
- added P6: Pad, hellen-one-common:PAD-TH, F.Cu at (171.4, 291.1)
- added P7: Pad, hellen-one-common:PAD-TH, F.Cu at (215.5, 313.1)
- added P8: Pad, hellen-one-common:PAD-TH, F.Cu at (215.5, 317.8)
- added Q10: ISL9V3040D3ST, Package_TO_SOT_SMD:TO-252-2, F.Cu at (155.0, 295.6)
- added Q11: ISL9V3040D3ST, Package_TO_SOT_SMD:TO-252-2, F.Cu at (155.0, 302.6)
- added Q12: ISL9V3040D3ST, Package_TO_SOT_SMD:TO-252-2, F.Cu at (155.0, 309.6)
- added Q7: ISL9V3040D3ST, Package_TO_SOT_SMD:TO-252-2, F.Cu at (155.0, 274.6)
- added Q8: ISL9V3040D3ST, Package_TO_SOT_SMD:TO-252-2, F.Cu at (155.0, 281.6)
- added Q9: ISL9V3040D3ST, Package_TO_SOT_SMD:TO-252-2, F.Cu at (155.0, 288.6)
- added R1: 4.7k, hellen-one-common:R0603, F.Cu at (167.2, 257.2)
- added R10: 4.7k, hellen-one-common:R0603, F.Cu at (160.9, 264.7)
- added R11: 4.7k, hellen-one-common:R0603, F.Cu at (162.5, 258.8)
- added R12: 4.7k, hellen-one-common:R0603, B.Cu at (162.6, 260.4)
- added R13: 4.7k, hellen-one-common:R0603, B.Cu at (162.6, 263.8)
- added R14: 4.7k, hellen-one-common:R0603, F.Cu at (155.9, 328.7)
- added R15: 4.7k, hellen-one-common:R0603, B.Cu at (134.8, 247.3)
- added R16: 4.7k, hellen-one-common:R0603, B.Cu at (137.4, 247.3)
- added R17: 22, hellen-one-common:R0603, B.Cu at (160.8, 274.7)
- added R18: 22, hellen-one-common:R0603, B.Cu at (160.8, 281.7)
- added R19: 22, hellen-one-common:R0603, B.Cu at (160.8, 288.7)
- added R2: 33k, hellen-one-common:R0603, B.Cu at (148.3, 316.1)
- added R20: 0, Resistor_SMD:R_2512_6332Metric, B.Cu at (156.2, 274.7)
- added R21: 0, Resistor_SMD:R_2512_6332Metric, B.Cu at (156.2, 281.7)
- added R22: 0, Resistor_SMD:R_2512_6332Metric, B.Cu at (156.2, 288.7)
- added R23: 22, hellen-one-common:R0603, B.Cu at (160.8, 295.7)
- added R24: 22, hellen-one-common:R0603, B.Cu at (160.8, 302.7)
- added R25: 22, hellen-one-common:R0603, B.Cu at (160.8, 309.7)
- added R26: 0, Resistor_SMD:R_2512_6332Metric, B.Cu at (156.2, 295.7)
- added R27: 0, Resistor_SMD:R_2512_6332Metric, B.Cu at (156.2, 302.7)
- added R28: 0, Resistor_SMD:R_2512_6332Metric, B.Cu at (156.2, 309.7)
- added R29: 4.7k, hellen-one-common:R0603, B.Cu at (136.6, 295.3)
- added R3: 6.8k, hellen-one-common:R0603, B.Cu at (148.3, 319.1)
- added R30: 4.7k, hellen-one-common:R0603, B.Cu at (168.5, 311.0)
- added R31: 4.7k, hellen-one-common:R0603, B.Cu at (134.9, 295.3)
- added R32: 4.7k, hellen-one-common:R0603, B.Cu at (166.2, 308.7)
- added R33: 4.7k, hellen-one-common:R0603, B.Cu at (164.3, 309.1)
- added R34: 4.7k, hellen-one-common:R0603, B.Cu at (138.2, 295.3)
- added R35: 10k, hellen-one-common:R0805, F.Cu at (227.1, 246.6)
- added R36: 10k, hellen-one-common:R0805, F.Cu at (227.1, 249.1)
- added R37: 10k, hellen-one-common:R0805, F.Cu at (227.1, 251.6)
- added R38: DNP, hellen-one-common:R0805, F.Cu at (230.5, 246.6)
- added R39: DNP, hellen-one-common:R0805, F.Cu at (230.5, 249.1)
- added R4: Jumper-Pad-Pad, hellen-one-common:PAD-0805-PAD, F.Cu at (175.8, 332.6)
- added R40: DNP, hellen-one-common:R0805, F.Cu at (230.5, 251.6)
- added R5: 0, hellen-one-common:R0603, B.Cu at (189.2, 275.3)
- added R6: 0, hellen-one-common:R0603, B.Cu at (209.9, 266.3)
- added R7: 5.6k, hellen-one-common:R0603, B.Cu at (181.3, 332.8)
- added R8: 5.6k, hellen-one-common:R0603, B.Cu at (183.8, 332.8)
- added R9: 4.7k, hellen-one-common:R0603, F.Cu at (149.0, 319.2)
- added U1: TLE9201SG, Package_SO:Infineon_PG-DSO-12-11, F.Cu at (141.3, 319.6)
- added U10: VNLD5160TR-E, Package_SO:SOIC-8_3.9x4.9mm_P1.27mm, B.Cu at (135.5, 277.7)
- added U11: VNLD5160TR-E, Package_SO:SOIC-8_3.9x4.9mm_P1.27mm, B.Cu at (135.5, 286.2)
- added U2: TLE9201SG, Package_SO:Infineon_PG-DSO-12-11, F.Cu at (147.9, 329.1)
- added U3: MPX4/MPXH6400_MAP, kicad6-libraries:MPX-4_MAP, F.Cu at (208.3, 273.1)
- added U4: MAX31855KASA, Package_SO:SOIC-8_3.9x4.9mm_P1.27mm, B.Cu at (187.8, 265.3)
- added U5: JDY-33, kicad6-libraries:JDY-33, F.Cu at (225.0, 316.0)
- added U6: VNLD5160TR-E, Package_SO:SOIC-8_3.9x4.9mm_P1.27mm, B.Cu at (136.7, 252.9)
- added U7: VNLD5160TR-E, Package_SO:SOIC-8_3.9x4.9mm_P1.27mm, F.Cu at (157.6, 260.3)
- added U8: VNLD5160TR-E, Package_SO:SOIC-8_3.9x4.9mm_P1.27mm, B.Cu at (157.6, 261.6)
- added U9: VNLD5160TR-E, Package_SO:SOIC-8_3.9x4.9mm_P1.27mm, B.Cu at (135.5, 268.9)
Routing:
- net (no net): track 0.00 -> 5262.1 mm, vias 0 -> 122
- net +12V_RAW: track 0.00 -> 250.7 mm, vias 0 -> 2
- net +5VP: track 0.00 -> 199.7 mm, vias 0 -> 3
- net +5VA: track 0.00 -> 171.8 mm, vias 0 -> 6
- net /CAN+: track 0.00 -> 102.6 mm
- net /CAN-: track 0.00 -> 100.8 mm
- net +5V: track 0.00 -> 45.9 mm, vias 0 -> 1
- net unconnected-(P1-Pad24): track 0.00 -> 43.1 mm
- net /IN_VIGN: track 0.00 -> 6.27 mm
- net GND: track 0.00 -> 1.50 mm, vias 0 -> 229
- added copper zone on B.Cu, net (none)
Other:
- board size 164 x 118 mm -> 186.6 x 344.8 mm
- board text added: "+ EGT -"
- board text added: "1"
- board text added: "10"
- board text added: "11"
- board text added: "12"
- board text added: "12V"
- board text added: "16"
- board text added: "18"
- board text added: "20"
- board text added: "3"
- board text added: "3.3"
- board text added: "4"
- board text added: "5"
- board text added: "5V"
- board text added: "6"
- board text added: "8"
- board text added: "9"
- board text added: "9924+"
- board text added: "9924-"
- board text added: "A"
- board text added: "AUX1"
- board text added: "AUX2"
- board text added: "AUX3"
- board text added: "Always looking for C/C++/PHP/Java developers https://rusefi.com/s/mission"
- board text added: "B"
- board text added: "BT1"
- board text added: "BT2"
- board text added: "BT3"
- board text added: "BTN1"
- board text added: "BTN2"
- board text added: "BTN3"
- board text added: "C"
- board text added: "CAN2"
- board text added: "CLT"
- board text added: "COMMUNITY SUPPORT ECU"
- board text added: "D"
- board text added: "DC1+"
- board text added: "DC1-"
- board text added: "DC2+"
- board text added: "DC2-"
- board text added: "DISCRETE+"
- board text added: "DISCRETE-"
- board text added: "DOWN"
- board text added: "E"
- board text added: "FLEX"
- board text added: "G"
- board text added: "G G + - V"
- board text added: "GND"
- board text added: "GNDA"
- board text added: "H"
- board text added: "H CAN L"
- board text added: "HALL1"
- board text added: "HALL2"
- board text added: "HALL3"
- board text added: "Heater"
- board text added: "IAT"
- board text added: "IGN1"
- board text added: "IGN2"
- board text added: "IGN3"
- board text added: "IGN4"
- board text added: "IGN5"
- board text added: "IGN6"
- board text added: "INJ1"
- board text added: "INJ2"
- board text added: "INJ3"
- board text added: "INJ4"
- board text added: "INJ5"
- board text added: "INJ6"
- board text added: "Ignition logic level outputs by default to control dumb coils remove R20-R22, R26-R28 and populate Q7-Q12"
- board text added: "Ip"
- board text added: "KNOCK"
- board text added: "L"
- board text added: "L CAN H"
- board text added: "LS1"
- board text added: "LS2"
- board text added: "LS3"
- board text added: "LS4"
- board text added: "LSH1"
- board text added: "LSH2"
- board text added: "MAP"
- board text added: "PPS1"
- board text added: "PPS2"
- board text added: "Rtrim"
- board text added: "SWD: R D G C V"
- board text added: "TPS1"
- board text added: "TPS2"
- board text added: "To enable Hall mode on VR9924-, populate R1"
- board text added: "UAEFI rev. E"
- board text added: "UART2 RX TX"
- board text added: "UP"
- board text added: "USB"
- board text added: "Un"
- board text added: "VIGN"
- board text added: "VR 9924 DISCR"
- board text added: "Vm"
- board text added: "WBO"
- board text added: "https://rusefi.com/s/uaefi"

Commit message: wewe
Parts:
- moved U1 319.1 mm to (360.0, 87.3)
- moved U2 314.4 mm to (360.0, 97.0)
- moved C10 305.9 mm to (364.5, 109.7)
- moved C5 305.9 mm to (364.5, 105.7)
- moved C4 305.7 mm to (362.2, 105.7)
- moved C9 305.7 mm to (362.2, 109.7)
- moved C3 305.5 mm to (360.0, 105.7)
- moved C8 305.5 mm to (360.0, 109.7)
- moved C2 305.4 mm to (357.7, 105.7)
- moved C7 305.4 mm to (357.7, 109.7)
- moved C1 305.2 mm to (355.5, 105.7)
- moved C6 305.2 mm to (355.5, 109.7)
- moved C18 302.3 mm to (364.5, 113.7)
- moved C23 302.3 mm to (364.5, 117.7)
- moved C17 302.1 mm to (362.2, 113.7)
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Routing:
- net (no net): track 5262.1 -> 0.00 mm, vias 122 -> 0
- net +12V_RAW: track 250.7 -> 0.00 mm, vias 2 -> 0
- net +5VP: track 199.7 -> 0.00 mm, vias 3 -> 0
- net +5VA: track 171.8 -> 0.00 mm, vias 6 -> 0
- net /CAN+: track 102.6 -> 0.00 mm
- net /CAN-: track 100.8 -> 0.00 mm
- net +5V: track 45.9 -> 0.00 mm, vias 1 -> 0
- net unconnected-(P1-Pad24): track 43.1 -> 0.00 mm
- net /IN_VIGN: track 6.27 -> 0.00 mm
- net GND: track 1.50 -> 0.00 mm, vias 229 -> 0
- removed copper zone on B.Cu, net (none)
Other:
- board size 186.6 x 344.8 mm -> 164 x 118 mm
- board text removed: "+ EGT -"
- board text removed: "1"
- board text removed: "10"
- board text removed: "11"
- board text removed: "12"
- board text removed: "12V"
- board text removed: "16"
- board text removed: "18"
- board text removed: "20"
- board text removed: "3"
- board text removed: "3.3"
- board text removed: "4"
- board text removed: "5"
- board text removed: "5V"
- board text removed: "6"
- board text removed: "8"
- board text removed: "9"
- board text removed: "9924+"
- board text removed: "9924-"
- board text removed: "A"
- board text removed: "AUX1"
- board text removed: "AUX2"
- board text removed: "AUX3"
- board text removed: "Always looking for C/C++/PHP/Java developers https://rusefi.com/s/mission"
- board text removed: "B"
- board text removed: "BT1"
- board text removed: "BT2"
- board text removed: "BT3"
- board text removed: "BTN1"
- board text removed: "BTN2"
- board text removed: "BTN3"
- board text removed: "C"
- board text removed: "CAN2"
- board text removed: "CLT"
- board text removed: "COMMUNITY SUPPORT ECU"
- board text removed: "D"
- board text removed: "DC1+"
- board text removed: "DC1-"
- board text removed: "DC2+"
- board text removed: "DC2-"
- board text removed: "DISCRETE+"
- board text removed: "DISCRETE-"
- board text removed: "DOWN"
- board text removed: "E"
- board text removed: "FLEX"
- board text removed: "G"
- board text removed: "G G + - V"
- board text removed: "GND"
- board text removed: "GNDA"
- board text removed: "H"
- board text removed: "H CAN L"
- board text removed: "HALL1"
- board text removed: "HALL2"
- board text removed: "HALL3"
- board text removed: "Heater"
- board text removed: "IAT"
- board text removed: "IGN1"
- board text removed: "IGN2"
- board text removed: "IGN3"
- board text removed: "IGN4"
- board text removed: "IGN5"
- board text removed: "IGN6"
- board text removed: "INJ1"
- board text removed: "INJ2"
- board text removed: "INJ3"
- board text removed: "INJ4"
- board text removed: "INJ5"
- board text removed: "INJ6"
- board text removed: "Ignition logic level outputs by default to control dumb coils remove R20-R22, R26-R28 and populate Q7-Q12"
- board text removed: "Ip"
- board text removed: "KNOCK"
- board text removed: "L"
- board text removed: "L CAN H"
- board text removed: "LS1"
- board text removed: "LS2"
- board text removed: "LS3"
- board text removed: "LS4"
- board text removed: "LSH1"
- board text removed: "LSH2"
- board text removed: "MAP"
- board text removed: "PPS1"
- board text removed: "PPS2"
- board text removed: "Rtrim"
- board text removed: "SWD: R D G C V"
- board text removed: "TPS1"
- board text removed: "TPS2"
- board text removed: "To enable Hall mode on VR9924-, populate R1"
- board text removed: "UAEFI rev. E"
- board text removed: "UART2 RX TX"
- board text removed: "UP"
- board text removed: "USB"
- board text removed: "Un"
- board text removed: "VIGN"
- board text removed: "VR 9924 DISCR"
- board text removed: "Vm"
- board text removed: "WBO"
- board text removed: "https://rusefi.com/s/uaefi"

Commit message: wewewe
Parts:
- removed G1: RUSEFI_LOGO, kicad6-libraries:rusefi_logo
- removed G2: LOGO, hellen-one-common:LOGO
- removed G3: PROTO_AREA, hellen-one-common:PROTO_AREA
- removed the G4 at (347.7, 115.4)
- removed H1, H2, H3, H4: M3, MountingHole:MountingHole_3.2mm_M3_Pad_Via
- removed J10: 5569-16A2, Connector_Molex:Molex_Mini-Fit_Jr_5569-16A2_2x08_P4.20mm_Horizontal
- removed J2: 5569-20A2, Connector_Molex:Molex_Mini-Fit_Jr_5569-20A2_2x10_P4.20mm_Horizontal
- moved Q12 237.0 mm to (90.5, 30.0), turned to 90 degrees
- moved Q11 226.6 mm to (97.5, 30.0), turned to 90 degrees
- moved Q10 216.4 mm to (104.5, 30.0), turned to 90 degrees
- moved Q9 206.1 mm to (111.5, 30.0), turned to 90 degrees
- moved U1 205.6 mm to (162.9, 29.1)
- moved U2 204.8 mm to (163.0, 41.0)
- moved M5 203.6 mm to (189.4, 52.2)
- moved Q8 195.9 mm to (118.5, 30.0), turned to 90 degrees
- moved U3 195.4 mm to (154.3, 76.6)
- moved U5 187.1 mm to (180.8, 75.2)
- moved Q7 185.8 mm to (125.5, 30.0), turned to 90 degrees
- moved M6 161.2 mm to (132.9, 56.6)
- moved P1 139.4 mm to (194.8, 69.1), turned to 180 degrees
- moved J3 115.0 mm to (371.2, 118.8)
- moved G4 106.2 mm to (143.2, 101.7), turned to 0 degrees
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Routing:
- net (no net): track 0.00 -> 5262.1 mm, vias 0 -> 122
- net +12V_RAW: track 0.00 -> 250.7 mm, vias 0 -> 2
- net +5VP: track 0.00 -> 199.7 mm, vias 0 -> 3
- net +5VA: track 0.00 -> 171.8 mm, vias 0 -> 6
- net /CAN+: track 0.00 -> 102.6 mm
- net /CAN-: track 0.00 -> 100.8 mm
- net +5V: track 0.00 -> 45.9 mm, vias 0 -> 1
- net /IN_VIGN: track 0.00 -> 6.27 mm
- net GND: track 0.00 -> 1.50 mm, vias 0 -> 229
- added copper zone on B.Cu, net (none)
- added copper zone on B.Cu, net GND
- added copper zone on F.Cu, net GND
- added copper zone on In1.Cu, net GND
- added copper zone on In2.Cu, net GND
Other:
- board size 164 x 118 mm -> 221.2 x 335.4 mm
- board text added: "+ EGT -"
- board text added: "1"
- board text added: "10"
- board text added: "11"
- board text added: "12"
- board text added: "12V"
- board text added: "16"
- board text added: "18"
- board text added: "20"
- board text added: "3"
- board text added: "3.3"
- board text added: "4"
- board text added: "5"
- board text added: "5V"
- board text added: "6"
- board text added: "8"
- board text added: "9"
- board text added: "9924+"
- board text added: "9924-"
- board text added: "A"
- board text added: "AUX1"
- board text added: "AUX2"
- board text added: "AUX3"
- board text added: "Always looking for C/C++/PHP/Java developers https://rusefi.com/s/mission"
- board text added: "B"
- board text added: "BT1"
- board text added: "BT2"
- board text added: "BT3"
- board text added: "BTN1"
- board text added: "BTN2"
- board text added: "BTN3"
- board text added: "C"
- board text added: "CAN2"
- board text added: "CLT"
- board text added: "COMMUNITY SUPPORT ECU"
- board text added: "D"
- board text added: "DC1+"
- board text added: "DC1-"
- board text added: "DC2+"
- board text added: "DC2-"
- board text added: "DISCRETE+"
- board text added: "DISCRETE-"
- board text added: "DOWN"
- board text added: "E"
- board text added: "FLEX"
- board text added: "G"
- board text added: "G G + - V"
- board text added: "GND"
- board text added: "GNDA"
- board text added: "H"
- board text added: "H CAN L"
- board text added: "HALL1"
- board text added: "HALL2"
- board text added: "HALL3"
- board text added: "Heater"
- board text added: "IAT"
- board text added: "IGN1"
- board text added: "IGN2"
- board text added: "IGN3"
- board text added: "IGN4"
- board text added: "IGN5"
- board text added: "IGN6"
- board text added: "INJ1"
- board text added: "INJ2"
- board text added: "INJ3"
- board text added: "INJ4"
- board text added: "INJ5"
- board text added: "INJ6"
- board text added: "Ignition logic level outputs by default to control dumb coils remove R20-R22, R26-R28 and populate Q7-Q12"
- board text added: "Ip"
- board text added: "KNOCK"
- board text added: "L"
- board text added: "L CAN H"
- board text added: "LS1"
- board text added: "LS2"
- board text added: "LS3"
- board text added: "LS4"
- board text added: "LSH1"
- board text added: "LSH2"
- board text added: "MAP"
- board text added: "PPS1"
- board text added: "PPS2"
- board text added: "Rtrim"
- board text added: "SWD: R D G C V"
- board text added: "TPS1"
- board text added: "TPS2"
- board text added: "To enable Hall mode on VR9924-, populate R1"
- board text added: "UAEFI rev. E"
- board text added: "UART2 RX TX"
- board text added: "UP"
- board text added: "USB"
- board text added: "Un"
- board text added: "VIGN"
- board text added: "VR 9924 DISCR"
- board text added: "Vm"
- board text added: "WBO"
- board text added: "https://rusefi.com/s/uaefi"

Commit message: wewewe
Parts:
- removed BT1: CR1220, kicad6-libraries:CR1220-2
- removed C1, C10, C14, C15, C16, C17, C18, C19, C2, C20, C21, C22, C23, C3, C4, C5, C6, C7, C8, C9: 10u, hellen-one-common:C0805
- removed C11, C24, C27, C29, C31, C33: 100n, hellen-one-common:C0603
- removed C12, C13, C25, C26, C28, C30: 10n, hellen-one-common:C0603
- removed C32: 1u, hellen-one-common:C0603
- removed D1: 1N4148WS, hellen-one-common:SOD-323
- removed D2, D3, D4, D5: B5819W, hellen-one-common:SOD-123
- removed D8: NUP2105L, Package_TO_SOT_SMD:SOT-23
- removed F1, F2, F3, F4: 12H1500D, hellen-one-common:PAD-1206-PAD
- removed F10, F5, F6, F7, F8, F9: 50mA, Fuse:Fuse_0603_1608Metric
- removed J1, J11, J12, J13, J14, J15, J16, J17, J18, J19, J20, J21, J22, J24: Conn_02x02_Odd_Even, Connector_PinSocket_2.54mm:PinSocket_2x02_P2.54mm_Vertical
- removed J3: 5569-06A2, Connector_Molex:Molex_Mini-Fit_Jr_5569-06A2_2x03_P4.20mm_Horizontal
- removed J4: 5569-08A2, Connector_Molex:Molex_Mini-Fit_Jr_5569-08A2_2x04_P4.20mm_Horizontal
- removed J5: 5569-18A2, Connector_Molex:Molex_Mini-Fit_Jr_5569-18A2_2x09_P4.20mm_Horizontal
- removed J9: USB_C, kicad6-libraries:USB_C
- removed L1, L2: 470R@100MHz, Inductor_SMD:L_0603_1608Metric
- removed M2: Module-knock-0.2, hellen-one-knock-0.2:knock
- removed P15, P16, P17, P18, P3, P4, P5, P6, P7, P8: Pad, hellen-one-common:PAD-TH
- removed R1, R10, R11, R12, R13, R14, R15, R16, R29, R30, R31, R32, R33, R34, R9: 4.7k, hellen-one-common:R0603
- removed R17, R18, R19, R23, R24, R25: 22, hellen-one-common:R0603
- removed R2: 33k, hellen-one-common:R0603
- removed R20, R21, R22, R26, R27, R28: 0, Resistor_SMD:R_2512_6332Metric
- removed R3: 6.8k, hellen-one-common:R0603
- removed R35, R36, R37: 10k, hellen-one-common:R0805
- removed R38, R39, R40: DNP, hellen-one-common:R0805
- removed R4: Jumper-Pad-Pad, hellen-one-common:PAD-0805-PAD
- removed R5, R6: 0, hellen-one-common:R0603
- removed R7, R8: 5.6k, hellen-one-common:R0603
- U10, U11, U4, U6, U8, U9: moved to F.Cu
- moved J7 300.7 mm to (81.0, 92.0), turned to 0 degrees
- moved J8 261.4 mm to (98.9, 89.8)
- moved M1 256.2 mm to (78.5, 77.3)
- moved P2 244.1 mm to (78.5, 81.6), turned to 90 degrees
- moved P1 240.6 mm to (78.5, 84.5), turned to 90 degrees
- moved M7 236.9 mm to (81.3, 85.9), turned to 0 degrees
- moved U4 235.5 mm to (114.6, 46.0), turned to 90 degrees
- moved J6 222.2 mm to (182.1, 56.5)
- moved U11 217.9 mm to (90.6, 46.0), turned to 90 degrees
- moved M3 213.1 mm to (132.3, 24.9)
- moved U10 208.7 mm to (96.6, 46.0), turned to 90 degrees
- moved U8 200.3 mm to (120.6, 46.1), turned to 90 degrees
- moved U9 199.6 mm to (102.5, 46.0), turned to 90 degrees
- moved U7 194.5 mm to (126.4, 46.1), turned to 90 degrees
- moved M4 192.8 mm to (144.2, 25.0)
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Routing:
- net (no net): track 5262.1 -> 0.00 mm, vias 122 -> 0
- net +12V_RAW: track 250.7 -> 0.00 mm, vias 2 -> 0
- net +5VP: track 199.7 -> 0.00 mm, vias 3 -> 0
- net +5VA: track 171.8 -> 0.00 mm, vias 6 -> 0
- net /CAN+: track 102.6 -> 0.00 mm
- net /CAN-: track 100.8 -> 0.00 mm
- net +5V: track 45.9 -> 0.00 mm, vias 1 -> 0
- net /IN_VIGN: track 6.27 -> 0.00 mm
- net GND: track 1.50 -> 0.00 mm, vias 229 -> 0
- net unconnected-(P1-Pad59): vias 31 -> 30
- removed copper zone on B.Cu, net (none)
- removed copper zone on B.Cu, net GND
- removed copper zone on F.Cu, net GND
- removed copper zone on In1.Cu, net GND
- removed copper zone on In2.Cu, net GND
Other:
- board size 221.2 x 335.4 mm -> 164 x 118 mm
- board text removed: "+ EGT -"
- board text removed: "1"
- board text removed: "10"
- board text removed: "11"
- board text removed: "12"
- board text removed: "12V"
- board text removed: "16"
- board text removed: "18"
- board text removed: "20"
- board text removed: "3"
- board text removed: "3.3"
- board text removed: "4"
- board text removed: "5"
- board text removed: "5V"
- board text removed: "6"
- board text removed: "8"
- board text removed: "9"
- board text removed: "9924+"
- board text removed: "9924-"
- board text removed: "A"
- board text removed: "AUX1"
- board text removed: "AUX2"
- board text removed: "AUX3"
- board text removed: "Always looking for C/C++/PHP/Java developers https://rusefi.com/s/mission"
- board text removed: "B"
- board text removed: "BT1"
- board text removed: "BT2"
- board text removed: "BT3"
- board text removed: "BTN1"
- board text removed: "BTN2"
- board text removed: "BTN3"
- board text removed: "C"
- board text removed: "CAN2"
- board text removed: "CLT"
- board text removed: "COMMUNITY SUPPORT ECU"
- board text removed: "D"
- board text removed: "DC1+"
- board text removed: "DC1-"
- board text removed: "DC2+"
- board text removed: "DC2-"
- board text removed: "DISCRETE+"
- board text removed: "DISCRETE-"
- board text removed: "DOWN"
- board text removed: "E"
- board text removed: "FLEX"
- board text removed: "G"
- board text removed: "G G + - V"
- board text removed: "GND"
- board text removed: "GNDA"
- board text removed: "H"
- board text removed: "H CAN L"
- board text removed: "HALL1"
- board text removed: "HALL2"
- board text removed: "HALL3"
- board text removed: "Heater"
- board text removed: "IAT"
- board text removed: "IGN1"
- board text removed: "IGN2"
- board text removed: "IGN3"
- board text removed: "IGN4"
- board text removed: "IGN5"
- board text removed: "IGN6"
- board text removed: "INJ1"
- board text removed: "INJ2"
- board text removed: "INJ3"
- board text removed: "INJ4"
- board text removed: "INJ5"
- board text removed: "INJ6"
- board text removed: "Ignition logic level outputs by default to control dumb coils remove R20-R22, R26-R28 and populate Q7-Q12"
- board text removed: "Ip"
- board text removed: "KNOCK"
- board text removed: "L"
- board text removed: "L CAN H"
- board text removed: "LS1"
- board text removed: "LS2"
- board text removed: "LS3"
- board text removed: "LS4"
- board text removed: "LSH1"
- board text removed: "LSH2"
- board text removed: "MAP"
- board text removed: "PPS1"
- board text removed: "PPS2"
- board text removed: "Rtrim"
- board text removed: "SWD: R D G C V"
- board text removed: "TPS1"
- board text removed: "TPS2"
- board text removed: "To enable Hall mode on VR9924-, populate R1"
- board text removed: "UAEFI rev. E"
- board text removed: "UART2 RX TX"
- board text removed: "UP"
- board text removed: "USB"
- board text removed: "Un"
- board text removed: "VIGN"
- board text removed: "VR 9924 DISCR"
- board text removed: "Vm"
- board text removed: "WBO"
- board text removed: "https://rusefi.com/s/uaefi"
